Commit message: Updated launch files to use uuv_name in preperation for having multiple vehicles.

File: bluerov2_standalone/catkin_ws/src/vandy_bluerov/urdf/base.xacro (robot description, xacro)
@@ -111,114 +111,115 @@
       voltage="16.8"
       update_rate="2.0"/>
-  </xacro:macro>
-<!-- FLS echosounder and Altimeter echosounder (rangefinder sonar) joints -->
-<joint name="sonar_front_joint" type="fixed">
-    <axis xyz="0 1 0" />
-    <origin rpy="0 0 0" xyz="0.5 0 0" />
-    <parent link="uuv0/base_link"/>
-    <child link="uuv0/base_sonar_front"/>
-</joint>
-<link name="uuv0/base_sonar_front">
-    <collision>
-      <origin xyz="0 0 0" rpy="0 0 0"/>
-      <geometry>
-        <box size="0.01 0.01 0.01"/>
-      </geometry>
-    </collision>
-    <visual>
-      <origin xyz="0 0 0" rpy="0 0 0"/>
-      <geometry>
-        <box size="0.01 0.01 0.01"/>
-      </geometry>
-    </visual>
-    <inertial>
-      <mass value="1e-5" />
-      <origin xyz="0 0 0" rpy="0 0 0"/>
-      <inertia ixx="1e-6" ixy="0" ixz="0" iyy="1e-6" iyz="0" izz="1e-6" />
-    </inertial>
- </link>
- <joint name="sonar_bottom_joint" type="fixed">
-    <axis xyz="0 1 0" />
-    <origin rpy="0 1.5708 0" xyz="0 0 -0.5" />
-    <parent link="uuv0/base_link"/>
-    <child link="uuv0/base_sonar_bottom"/>
-</joint>
-<link name="uuv0/base_sonar_bottom">
-    <collision>
-      <origin xyz="0 0 0" rpy="0 0 0"/>
-      <geometry>
-        <box size="0.01 0.01 0.01"/>
-      </geometry>
-    </collision>
-    <visual>
-      <origin xyz="0 0 0" rpy="0 0 0"/>
-      <geometry>
-        <box size="0.01 0.01 0.01"/>
-      </geometry>
-    </visual>
-    <inertial>
-      <mass value="1e-5" />
-      <origin xyz="0 0 0" rpy="0 0 0"/>
-      <inertia ixx="1e-6" ixy="0" ixz="0" iyy="1e-6" iyz="0" izz="1e-6" />
-    </inertial>
- </link>
-<joint name="camera_joint" type="fixed">
-    <axis xyz="0 0 0" />
-    <origin rpy="0 0 0" xyz="0.2 0 0.1" />
-    <parent link="uuv0/base_link"/>
-    <child link="uuv0/camera_link"/>
-  </joint>
-  <!-- Camera -->
-  <link name="uuv0/camera_link">
-    <collision>
-      <origin xyz="0 0 0" rpy="0 0 0"/>
-      <geometry>
-	      <box size="0.02 0.02 0.02"/>
-      </geometry>
-    </collision>
-    <visual>
-      <geometry>
-	      <box size="0.02 0.02 0.02"/>
-      </geometry>
-    </visual>
-  </link>
-  <!-- generate an optical frame http://www.ros.org/reps/rep-0103.html#suffix-frames
-      so that ros and opencv can operate on the camera frame correctly -->
-  <joint name="camera_optical_joint" type="fixed">
-  <!--   these values have to be these values otherwise the gazebo camera image
-        won't be aligned properly with the frame it is supposedly originating from -->
-    <origin xyz="0 0 0" rpy="0 0 0"/>
-    <parent link="uuv0/camera_link"/>
-    <child link="uuv0/camera_link_optical"/>
-  </joint>
-  <link name="uuv0/camera_link_optical">
-  </link>
-  <joint name="camera_depth_joint" type="fixed">
-  <!--   these values have to be these values otherwise the gazebo camera image
-        won't be aligned properly with the frame it is supposedly originating from -->
-    <origin xyz="0 0 0" rpy="0 0 0"/>
-    <parent link="uuv0/camera_link"/>
-    <child link="uuv0/camera_link_depth"/>
-  </joint>
-  <link name="uuv0/camera_link_depth">
-  </link>
-<!-- VU SSS -->
-<!-- Both side, splitted from SW -->
-<joint name="sss_joint" type="fixed">
-    <axis xyz="0 0 0" />
-    <origin rpy="1.5708 1.5708 1.5708" xyz="1.0 0.0 0" />
-    <parent link="uuv0/base_link"/>
-    <child link="uuv0/base_sss"/>
-</joint>
-<link name="uuv0/base_sss">
-</link>
-<!-- VU FLS -->
-<joint name="fis_joint" type="fixed">
-    <axis xyz="0 0 0" />
-    <origin rpy="0 0.7854 0" xyz="1 0 1" />
-    <parent link="uuv0/base_link"/>
-    <child link="uuv0/base_fis"/>
-</joint>
-<link name="uuv0/base_fis">
-</link>
+      <!-- </xacro:macro> -->
+    <!-- FLS echosounder and Altimeter echosounder (rangefinder sonar) joints -->
+    <joint name="sonar_front_joint" type="fixed">
+        <axis xyz="0 1 0" />
+        <origin rpy="0 0 0" xyz="0.5 0 0" />
+        <parent link="${namespace}/base_link"/>
+        <child link="${namespace}/base_sonar_front"/>
+    </joint>
+    <link name="${namespace}/base_sonar_front">
+        <collision>
+          <origin xyz="0 0 0" rpy="0 0 0"/>
+          <geometry>
+            <box size="0.01 0.01 0.01"/>
+          </geometry>
+        </collision>
+        <visual>
+          <origin xyz="0 0 0" rpy="0 0 0"/>
+          <geometry>
+            <box size="0.01 0.01 0.01"/>
+          </geometry>
+        </visual>
+        <inertial>
+          <mass value="1e-5" />
+          <origin xyz="0 0 0" rpy="0 0 0"/>
+          <inertia ixx="1e-6" ixy="0" ixz="0" iyy="1e-6" iyz="0" izz="1e-6" />
+        </inertial>
+    </link>
+    <joint name="sonar_bottom_joint" type="fixed">
+        <axis xyz="0 1 0" />
+        <origin rpy="0 1.5708 0" xyz="0 0 -0.5" />
+        <parent link="${namespace}/base_link"/>
+        <child link="${namespace}/base_sonar_bottom"/>
+    </joint>
+    <link name="${namespace}/base_sonar_bottom">
+        <collision>
+          <origin xyz="0 0 0" rpy="0 0 0"/>
+          <geometry>
+            <box size="0.01 0.01 0.01"/>
+          </geometry>
+        </collision>
+        <visual>
+          <origin xyz="0 0 0" rpy="0 0 0"/>
+          <geometry>
+            <box size="0.01 0.01 0.01"/>
+          </geometry>
+        </visual>
+        <inertial>
+          <mass value="1e-5" />
+          <origin xyz="0 0 0" rpy="0 0 0"/>
+          <inertia ixx="1e-6" ixy="0" ixz="0" iyy="1e-6" iyz="0" izz="1e-6" />
+        </inertial>
+    </link>
+    <joint name="camera_joint" type="fixed">
+        <axis xyz="0 0 0" />
+        <origin rpy="0 0 0" xyz="0.2 0 0.1" />
+        <parent link="${namespace}/base_link"/>
+        <child link="${namespace}/camera_link"/>
+      </joint>
+      <!-- Camera -->
+      <link name="${namespace}/camera_link">
+        <collision>
+          <origin xyz="0 0 0" rpy="0 0 0"/>
+          <geometry>
+            <box size="0.02 0.02 0.02"/>
+          </geometry>
+        </collision>
+        <visual>
+          <geometry>
+            <box size="0.02 0.02 0.02"/>
+          </geometry>
+        </visual>
+      </link>
+      <!-- generate an optical frame http://www.ros.org/reps/rep-0103.html#suffix-frames
+          so that ros and opencv can operate on the camera frame correctly -->
+      <joint name="camera_optical_joint" type="fixed">
+      <!--   these values have to be these values otherwise the gazebo camera image
+            won't be aligned properly with the frame it is supposedly originating from -->
+        <origin xyz="0 0 0" rpy="0 0 0"/>
+        <parent link="${namespace}/camera_link"/>
+        <child link="${namespace}/camera_link_optical"/>
+      </joint>
+      <link name="${namespace}/camera_link_optical">
+      </link>
+      <joint name="camera_depth_joint" type="fixed">
+      <!--   these values have to be these values otherwise the gazebo camera image
+            won't be aligned properly with the frame it is supposedly originating from -->
+        <origin xyz="0 0 0" rpy="0 0 0"/>
+        <parent link="${namespace}/camera_link"/>
+        <child link="${namespace}/camera_link_depth"/>
+      </joint>
+      <link name="${namespace}/camera_link_depth">
+      </link>
+    <!-- VU SSS -->
+    <!-- Both side, splitted from SW -->
+    <joint name="sss_joint" type="fixed">
+        <axis xyz="0 0 0" />
+        <origin rpy="1.5708 1.5708 1.5708" xyz="1.0 0.0 0" />
+        <parent link="${namespace}/base_link"/>
+        <child link="${namespace}/base_sss"/>
+    </joint>
+    <link name="${namespace}/base_sss">
+    </link>
+    <!-- VU FLS -->
+    <joint name="fis_joint" type="fixed">
+        <axis xyz="0 0 0" />
+        <origin rpy="0 0.7854 0" xyz="1 0 1" />
+        <parent link="${namespace}/base_link"/>
+        <child link="${namespace}/base_fis"/>
+    </joint>
+    <link name="${namespace}/base_fis">
+    </link>
+</xacro:macro>
 </robot>
