Commit message: changed namespace usage and modified sensor xacro files

File: bluerov2_standalone/catkin_ws/src/vandy_bluerov/robots/bluerov2_default.xacro (robot description, xacro)
@@ -14,5 +14,5 @@
     <xacro:arg name="noise" default="0.02"/>
     <!-- Create the bluerov2 -->
-    <xacro:bluerov2_base namespace="$(arg namespace)" noisy="false">
+    <xacro:bluerov2_base namespace="$(arg namespace)">
         <!-- The underwater object plugin is given as an input block parameter to
          allow the addition of external models of manipulator units -->

File: bluerov2_standalone/catkin_ws/src/vandy_bluerov/urdf/base.xacro (robot description, xacro)
@@ -47,5 +47,5 @@
   <!-- Vehicle macro -->
   <!-- <xacro:macro name="bluerov2_base" params="namespace debug *gazebo"> -->
-  <xacro:macro name="bluerov2_base" params="namespace noisy *gazebo">
+  <xacro:macro name="bluerov2_base" params="namespace *gazebo">
       <!-- Rigid body description of the base link -->
       <link name="${namespace}/base_link">
@@ -91,11 +91,60 @@
     <!-- Include the sensor modules: 3D Pose, IMU, Pressure, Camera -->
     <xacro:include filename="$(find vandy_bluerov)/urdf/bluerov_sensors.xacro">
-      <xacro:arg name="noisy" value="${noisy}"/>
     </xacro:include>
     <!-- Mount a Pose 3D sensor. -->
-    <xacro:default_pose_3d_macro
+    <!-- <xacro:default_pose_3d_macro
             namespace="${namespace}"
             parent_link="${namespace}/base_link"
-            inertial_reference_frame="world"/>
+            inertial_reference_frame="world"/> -->
+    <!-- <xacro:pose_3d_macro
+      namespace="${namespace}"
+      parent_link="${namespace}/base_link"
+      topic="pose_gt"
+      update_rate="20"
+      noise_sigma="0.0"
+      noise_amplitude="0.0"
+      suffix="enu"
+      reference_frame="world"
+      publish_ned_odom="false">
+      <origin xyz="0 0 0" rpy="0 0 0" />
+    </xacro:pose_3d_macro> -->
+    <joint name="pose_3d_joint" type="fixed">
+        <axis xyz="0 0 0" />
+        <origin rpy="0 0 0" xyz="0 0 0" />
+        <parent link="${namespace}/base_link"/>
+        <child link="${namespace}/pose_link"/>
+    </joint>
+    <link name="${namespace}/pose_link">
+        <collision>
+          <origin xyz="0 0 0" rpy="0 0 0"/>
+          <geometry>
+            <box size="0. 0 0"/>
+          </geometry>
+        </collision>
+        <visual>
+          <origin xyz="0 0 0" rpy="0 0 0"/>
+          <geometry>
+            <box size="0 0 0"/>
+          </geometry>
+        </visual>
+        <inertial>
+          <mass value="1e-5" />
+          <origin xyz="0 0 0" rpy="0 0 0"/>
+          <inertia ixx="1e-6" ixy="0" ixz="0" iyy="1e-6" iyz="0" izz="1e-6" />
+        </inertial>
+    </link>
+    <!-- Mount a ENU 3D pose sensor -->
+    <xacro:pose_3d_macro
+      namespace="${namespace}"
+      parent_link="${namespace}/pose_link"
+      topic="pose_gt"
+      update_rate="20"
+      noise_sigma="0.0"
+      noise_amplitude="0.0"
+      suffix=""
+      reference_frame="world"
+      publish_ned_odom="false">
+      <origin xyz="0 0 0" rpy="0 0 0" />
+    </xacro:pose_3d_macro>
     <!-- TODO: Parametrize the battery unit -->
     <xacro:basic_linear_battery_macro

File: bluerov2_standalone/catkin_ws/src/vandy_bluerov/urdf/bluerov_sensors.xacro (robot description, xacro)
@@ -13,13 +13,4 @@
 -->
 <robot xmlns:xacro="http://www.ros.org/wiki/xacro">
-    <xacro:arg name="noisy" default="true"/>
-    <!-- Mount a noisy 3D pose sensor -->
-        <!-- Add pose_gt with Gaussian noise -->
-        <xacro:pose_3d_sensor_ned namespace="$(arg namespace)"
-                                  suffix="noisy"
-                                  parent_link="$(arg namespace)/base_link"
-                                  gaussian_noise_sigma="0.10"
-                                  gaussian_noise_amplitude="1.0"
-                                  topic="pose_gt_noisy"/>
     <!-- DVL sensor -->
     <xacro:dvl_plugin_macro
@@ -69,17 +60,7 @@
             topic="${namespace}/pressure/state"/> -->
     <!-- IMU  -->
-    <xacro:if value="${noisy == 'false'}">
-        <xacro:default_imu_ned namespace="${namespace}" parent_link="${namespace}/base_link">
-            <origin xyz="0 0 0" rpy="0 0 0"/>
-        </xacro:default_imu_ned>
-    </xacro:if>
-    <!-- IMU  with thruster blade failure -->
-    <xacro:if value="${noisy == 'true'}">
-        <xacro:thruster_blade_fail_imu_ned namespace="$(arg namespace)"
-                                           parent_link="$(arg namespace)/base_link"
-                                           thruster_blade_failure="$(arg thruster_blade_failure)">
-            <origin xyz="0 0 0" rpy="0 0 0"/>
-        </xacro:thruster_blade_fail_imu_ned>
-    </xacro:if>
+    <xacro:default_imu_ned namespace="${namespace}" parent_link="${namespace}/base_link">
+        <origin xyz="0 0 0" rpy="0 0 0"/>
+    </xacro:default_imu_ned>
     <!-- <xacro:switchable_battery_consumer_macro
             link_name="${namespace}/imu_link"

File: bluerov2_standalone/catkin_ws/src/vandy_bluerov/urdf/sensor_snippets.xacro (robot description, xacro)
@@ -64,18 +64,3 @@
      </xacro:if>
   </xacro:macro>
-  <xacro:macro name="pose_3d_sensor_ned" params="namespace suffix parent_link
-    gaussian_noise_sigma gaussian_noise_amplitude topic">
-    <xacro:pose_3d_macro
-      namespace="${namespace}"
-      parent_link="${parent_link}"
-      topic="${topic}"
-      update_rate="20"
-      noise_sigma="${gaussian_noise_sigma}"
-      noise_amplitude="${gaussian_noise_amplitude}"
-      suffix="${suffix}"
-      reference_frame="world_ned"
-      publish_ned_odom="true">
-      <origin xyz="0 0 0" rpy="0 0 0" />
-    </xacro:pose_3d_macro>
-  </xacro:macro>
 </robot>

Commit message: updated sonar as macro to add namespace.

File: bluerov2_standalone/catkin_ws/src/vandy_bluerov/robots/bluerov2_default.xacro (robot description, xacro)
@@ -7,7 +7,7 @@
     <xacro:arg name="thruster_blade_failure" default="false"/>
     <!-- Include the ROV macro file xacro:bluerov2_base -->
+    <xacro:include filename="$(find vandy_bluerov)/urdf/gazebo.xacro"/>
     <xacro:include filename="$(find vandy_bluerov)/urdf/base.xacro"/>
     <!-- Hydrodynamic and hydrostatic parameters for the vehicle xacro:macro bluerov2_hydro_model -->
-    <xacro:include filename="$(find vandy_bluerov)/urdf/gazebo.xacro"/>
     <xacro:include filename="$(find uuv_sensor_ros_plugins)/urdf/sensor_snippets.xacro"/>
     <xacro:include filename="$(find vandy_bluerov)/urdf/sensor_snippets.xacro"/>
@@ -34,4 +34,132 @@
         </gazebo>
     </xacro:bluerov2_base>
+      <!-- FLS echosounder and Altimeter echosounder (rangefinder sonar) joints -->
+    <gazebo reference="$(arg namespace)/base_sonar_front">
+      <xacro:blueorv2_base_sonar_front namespace="$(arg namespace)"/>
+    </gazebo>
+    <joint name="sonar_front_joint" type="fixed">
+        <axis xyz="0 1 0" />
+        <origin rpy="0 0 0" xyz="0.5 0 0" />
+        <parent link="$(arg namespace)/base_link"/>
+        <child link="$(arg namespace)/base_sonar_front"/>
+    </joint>
+    <link name="$(arg namespace)/base_sonar_front">
+        <collision>
+          <origin xyz="0 0 0" rpy="0 0 0"/>
+          <geometry>
+            <box size="0.01 0.01 0.01"/>
+          </geometry>
+        </collision>
+        <visual>
+          <origin xyz="0 0 0" rpy="0 0 0"/>
+          <geometry>
+            <box size="0.01 0.01 0.01"/>
+          </geometry>
+        </visual>
+        <inertial>
+          <mass value="1e-5" />
+          <origin xyz="0 0 0" rpy="0 0 0"/>
+          <inertia ixx="1e-6" ixy="0" ixz="0" iyy="1e-6" iyz="0" izz="1e-6" />
+        </inertial>
+    </link>
+    <gazebo reference="$(arg namespace)/base_sonar_bottom">
+      <xacro:bluerov2_base_sonar_bottom namespace="$(arg namespace)"/>
+    </gazebo>
+    <joint name="sonar_bottom_joint" type="fixed">
+        <axis xyz="0 1 0" />
+        <origin rpy="0 1.5708 0" xyz="0 0 -0.5" />
+        <parent link="$(arg namespace)/base_link"/>
+        <child link="$(arg namespace)/base_sonar_bottom"/>
+    </joint>
+    <link name="$(arg namespace)/base_sonar_bottom">
+        <collision>
+          <origin xyz="0 0 0" rpy="0 0 0"/>
+          <geometry>
+            <box size="0.01 0.01 0.01"/>
+          </geometry>
+        </collision>
+        <visual>
+          <origin xyz="0 0 0" rpy="0 0 0"/>
+          <geometry>
+            <box size="0.01 0.01 0.01"/>
+          </geometry>
+        </visual>
+        <inertial>
+          <mass value="1e-5" />
+          <origin xyz="0 0 0" rpy="0 0 0"/>
+          <inertia ixx="1e-6" ixy="0" ixz="0" iyy="1e-6" iyz="0" izz="1e-6" />
+        </inertial>
+    </link>
+    <joint name="camera_joint" type="fixed">
+        <axis xyz="0 0 0" />
+        <origin rpy="0 0 0" xyz="0.2 0 0.1" />
+        <parent link="$(arg namespace)/base_link"/>
+        <child link="$(arg namespace)/camera_link"/>
+      </joint>
+      <!-- Camera -->
+      <link name="$(arg namespace)/camera_link">
+        <collision>
+          <origin xyz="0 0 0" rpy="0 0 0"/>
+          <geometry>
+            <box size="0.02 0.02 0.02"/>
+          </geometry>
+        </collision>
+        <visual>
+          <geometry>
+            <box size="0.02 0.02 0.02"/>
+          </geometry>
+        </visual>
+      </link>
+      <!-- generate an optical frame http://www.ros.org/reps/rep-0103.html#suffix-frames
+          so that ros and opencv can operate on the camera frame correctly -->
+      <!-- <gazebo reference="$(arg namespace)/camera_link_optical">
+        <xacro:bluerov2_camera_link_optical namespace="$(arg namespace)"/>
+      </gazebo>
+      <joint name="camera_optical_joint" type="fixed"> -->
+      <!--   these values have to be these values otherwise the gazebo camera image
+            won't be aligned properly with the frame it is supposedly originating from -->
+        <!-- <origin xyz="0 0 0" rpy="0 0 0"/>
+        <parent link="$(arg namespace)/camera_link"/>
+        <child link="$(arg namespace)/camera_link_optical"/>
+      </joint>
+      <link name="$(arg namespace)/camera_link_optical">
+      </link> -->
+      <!-- <gazebo reference="$(arg namespace)/camera_link_depth">
+        <xacro:bluerov2_camera_link_depth namespace="$(arg namespace)"/>
+      </gazebo>
+      <joint name="camera_depth_joint" type="fixed"> -->
+      <!--   these values have to be these values otherwise the gazebo camera image
+            won't be aligned properly with the frame it is supposedly originating from -->
+        <!-- <origin xyz="0 0 0" rpy="0 0 0"/>
+        <parent link="$(arg namespace)/camera_link"/>
+        <child link="$(arg namespace)/camera_link_depth"/>
+      </joint>
+      <link name="$(arg namespace)/camera_link_depth">
+      </link> -->
+    <!-- VU SSS -->
+    <!-- Both side, splitted from SW -->
+    <gazebo reference="$(arg namespace)/base_sss">
+    <xacro:blueorv2_sss namespace="$(arg namespace)"/>
+    </gazebo>
+    <joint name="sss_joint" type="fixed">
+        <axis xyz="0 0 0" />
+        <origin rpy="1.5708 1.5708 1.5708" xyz="1.0 0.0 0" />
+        <parent link="$(arg namespace)/base_link"/>
+        <child link="$(arg namespace)/base_sss"/>
+    </joint>
+    <link name="$(arg namespace)/base_sss">
+    </link>
+    <!-- VU FLS -->
+    <gazebo reference="$(arg namespace)/base_fis">
+      <xacro:blueorv2_fis namespace="$(arg namespace)"/>
+    </gazebo>
+    <joint name="fis_joint" type="fixed">
+        <axis xyz="0 0 0" />
+        <origin rpy="0 0.7854 0" xyz="1 0 1" />
+        <parent link="$(arg namespace)/base_link"/>
+        <child link="$(arg namespace)/base_fis"/>
+    </joint>
+    <link name="$(arg namespace)/base_fis">
+    </link>
     <!-- Joint state publisher plugin >
     <xacro:default_joint_state_publisher namespace="$(arg namespace)" update_rate="10"/-->

File: bluerov2_standalone/catkin_ws/src/vandy_bluerov/urdf/base.xacro (robot description, xacro)
@@ -160,115 +160,4 @@
       voltage="16.8"
       update_rate="2.0"/>
-      <!-- </xacro:macro> -->
-    <!-- FLS echosounder and Altimeter echosounder (rangefinder sonar) joints -->
-    <joint name="sonar_front_joint" type="fixed">
-        <axis xyz="0 1 0" />
-        <origin rpy="0 0 0" xyz="0.5 0 0" />
-        <parent link="${namespace}/base_link"/>
-        <child link="${namespace}/base_sonar_front"/>
-    </joint>
-    <link name="${namespace}/base_sonar_front">
-        <collision>
-          <origin xyz="0 0 0" rpy="0 0 0"/>
-          <geometry>
-            <box size="0.01 0.01 0.01"/>
-          </geometry>
-        </collision>
-        <visual>
-          <origin xyz="0 0 0" rpy="0 0 0"/>
-          <geometry>
-            <box size="0.01 0.01 0.01"/>
-          </geometry>
-        </visual>
-        <inertial>
-          <mass value="1e-5" />
-          <origin xyz="0 0 0" rpy="0 0 0"/>
-          <inertia ixx="1e-6" ixy="0" ixz="0" iyy="1e-6" iyz="0" izz="1e-6" />
-        </inertial>
-    </link>
-    <joint name="sonar_bottom_joint" type="fixed">
-        <axis xyz="0 1 0" />
-        <origin rpy="0 1.5708 0" xyz="0 0 -0.5" />
-        <parent link="${namespace}/base_link"/>
-        <child link="${namespace}/base_sonar_bottom"/>
-    </joint>
-    <link name="${namespace}/base_sonar_bottom">
-        <collision>
-          <origin xyz="0 0 0" rpy="0 0 0"/>
-          <geometry>
-            <box size="0.01 0.01 0.01"/>
-          </geometry>
-        </collision>
-        <visual>
-          <origin xyz="0 0 0" rpy="0 0 0"/>
-          <geometry>
-            <box size="0.01 0.01 0.01"/>
-          </geometry>
-        </visual>
-        <inertial>
-          <mass value="1e-5" />
-          <origin xyz="0 0 0" rpy="0 0 0"/>
-          <inertia ixx="1e-6" ixy="0" ixz="0" iyy="1e-6" iyz="0" izz="1e-6" />
-        </inertial>
-    </link>
-    <joint name="camera_joint" type="fixed">
-        <axis xyz="0 0 0" />
-        <origin rpy="0 0 0" xyz="0.2 0 0.1" />
-        <parent link="${namespace}/base_link"/>
-        <child link="${namespace}/camera_link"/>
-      </joint>
-      <!-- Camera -->
-      <link name="${namespace}/camera_link">
-        <collision>
-          <origin xyz="0 0 0" rpy="0 0 0"/>
-          <geometry>
-            <box size="0.02 0.02 0.02"/>
-          </geometry>
-        </collision>
-        <visual>
-          <geometry>
-            <box size="0.02 0.02 0.02"/>
-          </geometry>
-        </visual>
-      </link>
-      <!-- generate an optical frame http://www.ros.org/reps/rep-0103.html#suffix-frames
-          so that ros and opencv can operate on the camera frame correctly -->
-      <joint name="camera_optical_joint" type="fixed">
-      <!--   these values have to be these values otherwise the gazebo camera image
-            won't be aligned properly with the frame it is supposedly originating from -->
-        <origin xyz="0 0 0" rpy="0 0 0"/>
-        <parent link="${namespace}/camera_link"/>
-        <child link="${namespace}/camera_link_optical"/>
-      </joint>
-      <link name="${namespace}/camera_link_optical">
-      </link>
-      <joint name="camera_depth_joint" type="fixed">
-      <!--   these values have to be these values otherwise the gazebo camera image
-            won't be aligned properly with the frame it is supposedly originating from -->
-        <origin xyz="0 0 0" rpy="0 0 0"/>
-        <parent link="${namespace}/camera_link"/>
-        <child link="${namespace}/camera_link_depth"/>
-      </joint>
-      <link name="${namespace}/camera_link_depth">
-      </link>
-    <!-- VU SSS -->
-    <!-- Both side, splitted from SW -->
-    <joint name="sss_joint" type="fixed">
-        <axis xyz="0 0 0" />
-        <origin rpy="1.5708 1.5708 1.5708" xyz="1.0 0.0 0" />
-        <parent link="${namespace}/base_link"/>
-        <child link="${namespace}/base_sss"/>
-    </joint>
-    <link name="${namespace}/base_sss">
-    </link>
-    <!-- VU FLS -->
-    <joint name="fis_joint" type="fixed">
-        <axis xyz="0 0 0" />
-        <origin rpy="0 0.7854 0" xyz="1 0 1" />
-        <parent link="${namespace}/base_link"/>
-        <child link="${namespace}/base_fis"/>
-    </joint>
-    <link name="${namespace}/base_fis">
-    </link>
-</xacro:macro>
+  </xacro:macro>
 </robot>
