Commit message: updated sonar as macro to add namespace.

File: bluerov2_standalone/catkin_ws/src/vandy_bluerov/urdf/gazebo.xacro (robot description, xacro)
@@ -86,5 +86,7 @@
          </hydrodynamic_model>
       </link>
-      <gazebo reference="${namespace}/base_sonar_front">
+   </xacro:macro>
+      <!-- <gazebo reference="${namespace}/base_sonar_front">         -->
+      <xacro:macro name="blueorv2_base_sonar_front" params="namespace">
          <sensor type="ray" name="TeraRanger">
             <pose>0 0 0 0 0 0</pose>
@@ -122,6 +124,359 @@
             </plugin>
          </sensor>
-         </gazebo>
-      <gazebo reference="${namespace}/base_sonar_bottom">
+      <!-- <gazebo reference="${namespace}/base_sonar_front">         -->
+         <sensor type="ray" name="TeraRanger">
+            <pose>0 0 0 0 0 0</pose>
+            <visualize>false</visualize>
+            <update_rate>50</update_rate>
+            <ray>
+               <scan>
+                  <horizontal>
+                     <samples>10</samples>
+                     <resolution>1</resolution>
+                     <!-- 3 deg -->
+                     <min_angle>-0.0262</min_angle>
+                     <max_angle>0.0262</max_angle>
+                  </horizontal>
+                  <vertical>
+                     <samples>10</samples>
+                     <resolution>1</resolution>
+                     <!-- 3 deg -->
+                     <min_angle>-0.0262</min_angle>
+                     <max_angle>0.0262</max_angle>
+                  </vertical>
+               </scan>
+               <range>
+                  <min>0.5</min>
+                  <max>30</max>
+                  <resolution>0.15</resolution>
+               </range>
+            </ray>
+            <plugin filename="libgazebo_ros_range.so" name="gazebo_ros_range">
+               <gaussianNoise>0.005</gaussianNoise>
+               <alwaysOn>true</alwaysOn>
+               <updateRate>50</updateRate>
+               <topicName>/${namespace}/fls_sonar_0</topicName>
+               <frameName>${namespace}/base_fls_sonar</frameName>
+               <radiation>ULTRASOUND</radiation>
+               <fov>0.0524</fov>
+            </plugin>
+         </sensor>
+      <!-- </gazebo> -->
+      <!-- <gazebo reference="${namespace}/base_sonar_front">         -->
+         <sensor type="ray" name="TeraRanger">
+            <pose>0 0 0 0 0 0</pose>
+            <visualize>false</visualize>
+            <update_rate>50</update_rate>
+            <ray>
+               <scan>
+                  <horizontal>
+                     <samples>10</samples>
+                     <resolution>1</resolution>
+                     <!-- 3 deg -->
+                     <min_angle>-0.0524</min_angle>
+                     <max_angle>0</max_angle>
+                  </horizontal>
+                  <vertical>
+                     <samples>10</samples>
+                     <resolution>1</resolution>
+                     <!-- 3 deg -->
+                     <min_angle>-0.0262</min_angle>
+                     <max_angle>0.0262</max_angle>
+                  </vertical>
+               </scan>
+               <range>
+                  <min>0.5</min>
+                  <max>30</max>
+                  <resolution>0.15</resolution>
+               </range>
+            </ray>
+            <plugin filename="libgazebo_ros_range.so" name="gazebo_ros_range">
+               <gaussianNoise>0.005</gaussianNoise>
+               <alwaysOn>true</alwaysOn>
+               <updateRate>50</updateRate>
+               <topicName>/${namespace}/fls_sonar_1</topicName>
+               <frameName>${namespace}/base_fls_sonar</frameName>
+               <radiation>ULTRASOUND</radiation>
+               <fov>0.0524</fov>
+            </plugin>
+         </sensor>
+      <!-- </gazebo> -->
+      <!-- <gazebo reference="${namespace}/base_sonar_front">         -->
+         <sensor type="ray" name="TeraRanger">
+            <pose>0 0 0 0 0 0</pose>
+            <visualize>false</visualize>
+            <update_rate>50</update_rate>
+            <ray>
+               <scan>
+                  <horizontal>
+                     <samples>10</samples>
+                     <resolution>1</resolution>
+                     <!-- 3 deg -->
+                     <min_angle>-0</min_angle>
+                     <max_angle>0.0524</max_angle>
+                  </horizontal>
+                  <vertical>
+                     <samples>10</samples>
+                     <resolution>1</resolution>
+                     <!-- 3 deg -->
+                     <min_angle>-0.0262</min_angle>
+                     <max_angle>0.0262</max_angle>
+                  </vertical>
+               </scan>
+               <range>
+                  <min>0.5</min>
+                  <max>30</max>
+                  <resolution>0.15</resolution>
+               </range>
+            </ray>
+            <plugin filename="libgazebo_ros_range.so" name="gazebo_ros_range">
+               <gaussianNoise>0.005</gaussianNoise>
+               <alwaysOn>true</alwaysOn>
+               <updateRate>50</updateRate>
+               <topicName>/${namespace}/fls_sonar_2</topicName>
+               <frameName>${namespace}/base_fls_sonar</frameName>
+               <radiation>ULTRASOUND</radiation>
+               <fov>0.0524</fov>
+            </plugin>
+         </sensor>
+      <!-- </gazebo> -->
+      <!-- <gazebo reference="${namespace}/base_sonar_front">         -->
+         <sensor type="ray" name="TeraRanger">
+            <pose>0 0 0 0 0 0</pose>
+            <visualize>false</visualize>
+            <update_rate>50</update_rate>
+            <ray>
+               <scan>
+                  <horizontal>
+                     <samples>10</samples>
+                     <resolution>1</resolution>
+                     <!-- 3 deg -->
+                     <min_angle>-0.0262</min_angle>
+                     <max_angle>0.0262</max_angle>
+                  </horizontal>
+                  <vertical>
+                     <samples>10</samples>
+                     <resolution>1</resolution>
+                     <!-- 3 deg -->
+                     <min_angle>-0</min_angle>
+                     <max_angle>0.0524</max_angle>
+                  </vertical>
+               </scan>
+               <range>
+                  <min>0.5</min>
+                  <max>30</max>
+                  <resolution>0.15</resolution>
+               </range>
+            </ray>
+            <plugin filename="libgazebo_ros_range.so" name="gazebo_ros_range">
+               <gaussianNoise>0.005</gaussianNoise>
+               <alwaysOn>true</alwaysOn>
+               <updateRate>50</updateRate>
+               <topicName>/${namespace}/fls_sonar_3</topicName>
+               <frameName>${namespace}/base_fls_sonar</frameName>
+               <radiation>ULTRASOUND</radiation>
+               <fov>0.0524</fov>
+            </plugin>
+         </sensor>
+      <!-- </gazebo> -->
+      <!-- <gazebo reference="${namespace}/base_sonar_front">         -->
+         <sensor type="ray" name="TeraRanger">
+            <pose>0 0 0 0 0 0</pose>
+            <visualize>false</visualize>
+            <update_rate>50</update_rate>
+            <ray>
+               <scan>
+                  <horizontal>
+                     <samples>10</samples>
+                     <resolution>1</resolution>
+                     <!-- 3 deg -->
+                     <min_angle>-0.0262</min_angle>
+                     <max_angle>0.0262</max_angle>
+                  </horizontal>
+                  <vertical>
+                     <samples>10</samples>
+                     <resolution>1</resolution>
+                     <!-- 3 deg -->
+                     <min_angle>-0.0524</min_angle>
+                     <max_angle>0</max_angle>
+                  </vertical>
+               </scan>
+               <range>
+                  <min>0.5</min>
+                  <max>30</max>
+                  <resolution>0.15</resolution>
+               </range>
+            </ray>
+            <plugin filename="libgazebo_ros_range.so" name="gazebo_ros_range">
+               <gaussianNoise>0.005</gaussianNoise>
+               <alwaysOn>true</alwaysOn>
+               <updateRate>50</updateRate>
+               <topicName>/${namespace}/fls_sonar_4</topicName>
+               <frameName>${namespace}/base_fls_sonar</frameName>
+               <radiation>ULTRASOUND</radiation>
+               <fov>0.0524</fov>
+            </plugin>
+         </sensor>
+      <!-- </gazebo> -->
+      <!-- <gazebo reference="${namespace}/base_sonar_front">         -->
+         <sensor type="ray" name="TeraRanger">
+            <pose>0 0 0 0 0 0</pose>
+            <visualize>false</visualize>
+            <update_rate>50</update_rate>
+            <ray>
+               <scan>
+                  <horizontal>
+                     <samples>10</samples>
+                     <resolution>1</resolution>
+                     <!-- 3 deg -->
+                     <min_angle>-0.0524</min_angle>
+                     <max_angle>0</max_angle>
+                  </horizontal>
+                  <vertical>
+                     <samples>10</samples>
+                     <resolution>1</resolution>
+                     <!-- 3 deg -->
+                     <min_angle>-0.0524</min_angle>
+                     <max_angle>0</max_angle>
+                  </vertical>
+               </scan>
+               <range>
+                  <min>0.5</min>
+                  <max>30</max>
+                  <resolution>0.15</resolution>
+               </range>
+            </ray>
+            <plugin filename="libgazebo_ros_range.so" name="gazebo_ros_range">
+               <gaussianNoise>0.005</gaussianNoise>
+               <alwaysOn>true</alwaysOn>
+               <updateRate>50</updateRate>
+               <topicName>/${namespace}/fls_sonar_5</topicName>
+               <frameName>${namespace}/base_fls_sonar</frameName>
+               <radiation>ULTRASOUND</radiation>
+               <fov>0.0524</fov>
+            </plugin>
+         </sensor>
+      <!-- </gazebo> -->
+      <!-- <gazebo reference="${namespace}/base_sonar_front">         -->
+         <sensor type="ray" name="TeraRanger">
+            <pose>0 0 0 0 0 0</pose>
+            <visualize>false</visualize>
+            <update_rate>50</update_rate>
+            <ray>
+               <scan>
+                  <horizontal>
+                     <samples>10</samples>
+                     <resolution>1</resolution>
+                     <!-- 3 deg -->
+                     <min_angle>-0</min_angle>
+                     <max_angle>0.0524</max_angle>
+                  </horizontal>
+                  <vertical>
+                     <samples>10</samples>
+                     <resolution>1</resolution>
+                     <!-- 3 deg -->
+                     <min_angle>-0.0524</min_angle>
+                     <max_angle>0</max_angle>
+                  </vertical>
+               </scan>
+               <range>
+                  <min>0.5</min>
+                  <max>30</max>
+                  <resolution>0.15</resolution>
+               </range>
+            </ray>
+            <plugin filename="libgazebo_ros_range.so" name="gazebo_ros_range">
+               <gaussianNoise>0.005</gaussianNoise>
+               <alwaysOn>true</alwaysOn>
+               <updateRate>50</updateRate>
+               <topicName>/${namespace}/fls_sonar_6</topicName>
+               <frameName>${namespace}/base_fls_sonar</frameName>
+               <radiation>ULTRASOUND</radiation>
+               <fov>0.0524</fov>
+            </plugin>
+         </sensor>
+      <!-- </gazebo> -->
+      <!-- <gazebo reference="${namespace}/base_sonar_front">         -->
+         <sensor type="ray" name="TeraRanger">
+            <pose>0 0 0 0 0 0</pose>
+            <visualize>false</visualize>
+            <update_rate>50</update_rate>
+            <ray>
+               <scan>
+                  <horizontal>
+                     <samples>10</samples>
+                     <resolution>1</resolution>
+                     <!-- 3 deg -->
+                     <min_angle>-0.0524</min_angle>
+                     <max_angle>0</max_angle>
+                  </horizontal>
+                  <vertical>
+                     <samples>10</samples>
+                     <resolution>1</resolution>
+                     <!-- 3 deg -->
+                     <min_angle>-0</min_angle>
+                     <max_angle>0.0524</max_angle>
+                  </vertical>
+               </scan>
+               <range>
+                  <min>0.5</min>
+                  <max>30</max>
+                  <resolution>0.15</resolution>
+               </range>
+            </ray>
+            <plugin filename="libgazebo_ros_range.so" name="gazebo_ros_range">
+               <gaussianNoise>0.005</gaussianNoise>
+               <alwaysOn>true</alwaysOn>
+               <updateRate>50</updateRate>
+               <topicName>/${namespace}/fls_sonar_7</topicName>
+               <frameName>${namespace}/base_fls_sonar</frameName>
+               <radiation>ULTRASOUND</radiation>
+               <fov>0.0524</fov>
+            </plugin>
+         </sensor>
+      <!-- </gazebo> -->
+      <!-- <gazebo reference="${namespace}/base_sonar_front">         -->
+         <sensor type="ray" name="TeraRanger">
+            <pose>0 0 0 0 0 0</pose>
+            <visualize>false</visualize>
+            <update_rate>50</update_rate>
+            <ray>
+               <scan>
+                  <horizontal>
+                     <samples>10</samples>
+                     <resolution>1</resolution>
+                     <!-- 3 deg -->
+                     <min_angle>-0</min_angle>
+                     <max_angle>0.0524</max_angle>
+                  </horizontal>
+                  <vertical>
+                     <samples>10</samples>
+                     <resolution>1</resolution>
+                     <!-- 3 deg -->
+                     <min_angle>-0</min_angle>
+                     <max_angle>0.0524</max_angle>
+                  </vertical>
+               </scan>
+               <range>
+                  <min>0.5</min>
+                  <max>30</max>
+                  <resolution>0.15</resolution>
+               </range>
+            </ray>
+            <plugin filename="libgazebo_ros_range.so" name="gazebo_ros_range">
+               <gaussianNoise>0.005</gaussianNoise>
+               <alwaysOn>true</alwaysOn>
+               <updateRate>50</updateRate>
+               <topicName>/${namespace}/fls_sonar_8</topicName>
+               <frameName>${namespace}/base_fls_sonar</frameName>
+               <radiation>ULTRASOUND</radiation>
+               <fov>0.0524</fov>
+            </plugin>
+         </sensor>
+      <!-- </gazebo> -->
+         <!-- </gazebo> -->
+      </xacro:macro>
+      <!-- <gazebo reference="${namespace}/base_sonar_bottom">   -->
+      <xacro:macro name="bluerov2_base_sonar_bottom" params="namespace">
          <sensor type="ray" name="TeraRanger">
             <pose>0 0 0 0 0 0</pose>
@@ -159,6 +514,8 @@
             </plugin>
          </sensor>
-         </gazebo>
-      <gazebo reference="${namespace}/camera_link_optical">
+         </xacro:macro>
+         <!-- </gazebo> -->
+      <!-- <gazebo reference="${namespace}/camera_link_optical"> -->
+      <xacro:macro name="bluerov2_camera_link_optical" params="namespace">
          <sensor type="camera" name="camera_camera_sensor">
             <update_rate>30.0</update_rate>
@@ -199,47 +556,49 @@
             </plugin>
          </sensor>
-      </gazebo>
-      <gazebo reference="${namespace}/camera_link_depth">
-      <sensor name="${namespace}/camera_link_depth_camera" type="depth">
-         <update_rate>20</update_rate>
-         <camera>
-            <horizontal_fov>1.047198</horizontal_fov>
-            <image>
-            <width>640</width>
-            <height>480</height>
-            <format>R8G8B8</format>
-            </image>
-            <clip>
-            <near>0.05</near>
-            <far>100</far>
-            </clip>
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